File: SUSTAINA-Core-Board.brd (EAGLE design)
At the start: 120 x 70 mm, 67 parts, among them IC1 LTC4418IUF, M1 POWER-MONITOR-MODULE, M2 POWER-MONITOR-MODULE, M3 BUCK-BOOST-SWITCH-MODE-POWER-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, M4 POWER-MONITOR-MODULE, M5 POWER-MONITOR-MODULE, Q1 SUM110P06-08L-E3, Q2 SUM110P06-08L-E3, Q3 SUM110P06-08L-E3, Q4 SUM110P06-08L-E3, Q5 SUM110P06-08L-E3, Q6 SUM110P06-08L-E3

Commit message: Upload data for RoboCup2023 competition specifications
Parts:
- added LED5: Green, led:SML0603
- added R19: 2k, rcl:R0603
- C10, C9: value 0.1u -> 1u
- moved CH4 107.3 mm to (54.0, -20.3), turned to 90 degrees
- moved CH5 107.3 mm to (-54.0, -20.3), turned to 270 degrees
- moved CH8 4.55 mm to (-43.2, 11.7)
- moved C10 1.91 mm to (22.2, 6.35)
- moved C9 1.91 mm to (-22.2, 6.35)
- moved R13 1.91 mm to (-24.8, 6.35)
- moved R15 1.91 mm to (24.8, 6.35)
- moved R14 1.90 mm to (-19.7, 6.35)
- moved R16 1.90 mm to (19.7, 6.35)
- moved C5 1.27 mm to (23.5, -10.5), turned to 0 degrees
- moved C6 1.27 mm to (23.5, -2.22)
- moved Q1 1.27 mm to (29.8, -6.35)
- moved Q3 1.27 mm to (-29.8, -6.35)
- moved Q5 1.27 mm to (-29.8, 6.35)
- moved Q6 1.27 mm to (29.8, 6.35)
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Connections:
- net +ACTUATOR_POWER renamed +ACTR_PWR
- net +ACTUATOR_POWER_INPUT renamed +ACTR_PWR_INPUT
- net +ACTUATOR_SENSING renamed +ACTR_SENSING
- net +BATTERY_INPUT1 renamed +BATT_INPUT1
- net +BATTERY_INPUT1_FUSE renamed +BATT_INPUT1_FUSE
- net +BATTERY_INPUT2 renamed +BATT_INPUT2
- net +BATTERY_INPUT2_FUSE renamed +BATT_INPUT2_FUSE
- net +BATTERY_INPUT_SENSING1 renamed +BATT_INPUT_SENSING1
- net +BATTERY_INPUT_SENSING2 renamed +BATT_INPUT_SENSING2
- net +POWER_INPUT renamed +PWR_INPUT
- net +SBC_POWER renamed +SBC_PWR
- net +SBC_POWER_INPUT renamed +SBC_PWR_INPUT
- net +SBC_POWER_OUTPUT renamed +SBC_PWR_OUTPUT
- net GATE_ACTUATOR renamed GATE_ACTR
- net GATE_ACTUATOR_ renamed GATE_ACTR_
- new net LED_3V3: LED5.A, R19.1
- net +3V3: now also R19.2
- net GND: now also LED5.C
Routing:
- net GATE_ACTR_: track 57.6 -> 94.0 mm, vias 1 -> 2
- net GATE_SBC_: track 60.6 -> 95.7 mm, vias 5 -> 2
- net GND: track 33.0 -> 9.73 mm, vias 0 -> 5
- net I2C_SDA: track 235.1 -> 213.4 mm, vias 1 -> 2
- net +BATT_INPUT_SENSING2: track 65.7 -> 50.7 mm
- net I2C_SCL: track 223.3 -> 212.4 mm, vias 1 -> 2
- net +PWR_INPUT: track 73.2 -> 82.7 mm
- net VS2: track 24.9 -> 34.0 mm
- net G1: track 33.8 -> 42.9 mm
- net C-DM: track 92.6 -> 98.0 mm
- net D-DP: track 78.8 -> 74.1 mm
- net +3V3: track 218.7 -> 223.3 mm
- net A-DP: track 93.7 -> 89.8 mm
- net B-DP: track 59.2 -> 62.6 mm
- net +BATT_INPUT_SENSING1: track 57.0 -> 60.1 mm
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Other:
- board text added: "3V3"
- board text added: "3V3 >"
- board text added: "< Priority 1st Power Input"
- board text added: "< Priority 2nd Power Input"
- board text added: "A"
- board text added: "Actuator Power ON/OFF Switch"
- board text added: "Actuator Power Output >"
- board text added: "B"
- board text added: "Buck-Boost Switch Mode Power Supply Module"
- board text added: "C"
- board text added: "Connection Port to the Expansion Board"
- board text added: "D"
- board text added: "Fuse"
- board text added: "I2C"
- board text added: "NC"
- board text added: "Power Monitor Module"
- board text added: "Power Output >"
- board text added: "Power Supply Input"
- board text added: "RS-485 Channels"
- board text added: "SBC"
- board text added: "SBC Power ON/OFF Switch"
- board text added: "SCL"
- board text added: "SDA"
- board text added: "SUSTAINA Core Board Rev. 1 Designed by Masato Kubotera on June 12, 2023."
- board text added: "VIN"
- board text added: "VIN+"
- board text added: "VIN-"
- board text added: "VOUT"
- board text added: "Voltage Indicator"
- board text removed: "Actuator Switch"
- board text removed: "SBC Switch"
- board text removed: "SUSTAINA Core Board Rev. 1 Designed by Masato Kubotera on June 1, 2023."
- board text removed: "Voltmeter LCD"

Commit message: Solved the problem of not being able to use a switching power supply in Rev.1
Parts:
- C10, C9: value 1u -> 0.1u
- C5, C7: value 0.1u -> 1u
- R3, R6: value 1180k -> 18k
- R4, R7: value 34k -> 2k
- R5, R8: value 86.6k -> 1k
Changed lines of the file:
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@@
 <attribute name="NAME" x="-39.6875" y="1.27" size="0.8" layer="25" ratio="10" rot="R90" align="center"/>
 </element>
-<element name="C9" library="rcl" library_urn="urn:adsk.eagle:library:334" package="C0603" package3d_urn="urn:adsk.eagle:package:23616/2" value="1u" x="-22.225" y="6.35" smashed="yes" rot="R270">
+<element name="C9" library="rcl" library_urn="urn:adsk.eagle:library:334" package="C0603" package3d_urn="urn:adsk.eagle:package:23616/2" value="0.1u" x="-22.225" y="6.35" smashed="yes" rot="R270">
 <attribute name="NAME" x="-20.955" y="6.35" size="0.8" layer="25" ratio="10" rot="R270" align="center"/>
 <attribute name="POPULARITY" value="37" x="-94.615" y="-68.58" size="1.778" layer="27" rot="R270" display="off"/>
@@
 <attribute name="VALUE" x="22.86" y="6.985" size="1.27" layer="27" rot="R270"/>
 </element>
-<element name="C10" library="rcl" library_urn="urn:adsk.eagle:library:334" package="C0603" package3d_urn="urn:adsk.eagle:package:23616/2" value="1u" x="22.225" y="6.35" smashed="yes" rot="R90">
+<element name="C10" library="rcl" library_urn="urn:adsk.eagle:library:334" package="C0603" package3d_urn="urn:adsk.eagle:package:23616/2" value="0.1u" x="22.225" y="6.35" smashed="yes" rot="R90">
 <attribute name="NAME" x="20.955" y="6.35" size="0.8" layer="25" ratio="10" rot="R90" align="center"/>
 <attribute name="POPULARITY" value="37" x="12.065" y="-11.43" size="1.778" layer="27" rot="R90" display="off"/>
@@
 <attribute name="VALUE" x="4.445" y="-28.8925" size="1.27" layer="27"/>
 </element>
-<element name="C5" library="rcl" library_urn="urn:adsk.eagle:library:334" package="C0603" package3d_urn="urn:adsk.eagle:package:23616/2" value="0.1u" x="23.495" y="-10.4775" smashed="yes">
+<element name="C5" library="rcl" library_urn="urn:adsk.eagle:library:334" package="C0603" package3d_urn="urn:adsk.eagle:package:23616/2" value="1u" x="23.495" y="-10.4775" smashed="yes">
 <attribute name="NAME" x="23.495" y="-11.7475" size="0.8" layer="25" ratio="10" align="center"/>
 <attribute name="POPULARITY" value="37" x="23.495" y="-10.4775" size="1.778" layer="27" display="off"/>
@@
 <attribute name="VALUE" x="22.86" y="-12.3825" size="1.27" layer="27"/>
 </element>
-<element name="C7" library="rcl" library_urn="urn:adsk.eagle:library:334" package="C0603" package3d_urn="urn:adsk.eagle:package:23616/2" value="0.1u" x="-15.24" y="-13.0175" smashed="yes">
+<element name="C7" library="rcl" library_urn="urn:adsk.eagle:library:334" package="C0603" package3d_urn="urn:adsk.eagle:package:23616/2" value="1u" x="-15.24" y="-13.0175" smashed="yes">
 <attribute name="NAME" x="-15.24" y="-14.2875" size="0.8" layer="25" ratio="10" align="center"/>
 <attribute name="POPULARITY" value="37" x="-15.24" y="-13.0175" size="1.778" layer="27" display="off"/>
@@
 <attribute name="VALUE" x="-15.875" y="-14.9225" size="1.27" layer="27"/>
 </element>
-<element name="R3" library="rcl" library_urn="urn:adsk.eagle:library:334" package="R0603" package3d_urn="urn:adsk.eagle:package:23555/3" value="1180k" x="-6.35" y="-20.6375" smashed="yes" rot="R90">
+<element name="R3" library="rcl" library_urn="urn:adsk.eagle:library:334" package="R0603" package3d_urn="urn:adsk.eagle:package:23555/3" value="18k" x="-6.35" y="-20.6375" smashed="yes" rot="R90">
 <attribute name="NAME" x="-5.08" y="-20.6375" size="0.8" layer="25" ratio="10" rot="R90" align="center"/>
 <attribute name="POPULARITY" value="77" x="-6.35" y="-20.6375" size="1.778" layer="27" rot="R90" display="off"/>
@@
 <attribute name="VALUE" x="-4.445" y="-21.2725" size="1.27" layer="27" rot="R90"/>
 </element>
-<element name="R4" library="rcl" library_urn="urn:adsk.eagle:library:334" package="R0603" package3d_urn="urn:adsk.eagle:package:23555/3" value="34k" x="-3.81" y="-22.5425" smashed="yes" rot="R90">
+<element name="R4" library="rcl" library_urn="urn:adsk.eagle:library:334" package="R0603" package3d_urn="urn:adsk.eagle:package:23555/3" value="2k" x="-3.81" y="-22.5425" smashed="yes" rot="R90">
 <attribute name="NAME" x="-2.54" y="-22.5425" size="0.8" layer="25" ratio="10" rot="R90" align="center"/>
 <attribute name="POPULARITY" value="77" x="-3.81" y="-22.5425" size="1.778" layer="27" rot="R90" display="off"/>
@@
 <attribute name="VALUE" x="-1.905" y="-23.1775" size="1.27" layer="27" rot="R90"/>
 </element>
-<element name="R5" library="rcl" library_urn="urn:adsk.eagle:library:334" package="R0603" package3d_urn="urn:adsk.eagle:package:23555/3" value="86.6k" x="-6.35" y="-23.8125" smashed="yes" rot="R90">
+<element name="R5" library="rcl" library_urn="urn:adsk.eagle:library:334" package="R0603" package3d_urn="urn:adsk.eagle:package:23555/3" value="1k" x="-6.35" y="-23.8125" smashed="yes" rot="R90">
 <attribute name="NAME" x="-5.08" y="-23.8125" size="0.8" layer="25" ratio="10" rot="R90" align="center"/>
 <attribute name="POPULARITY" value="77" x="-6.35" y="-23.8125" size="1.778" layer="27" rot="R90" display="off"/>
@@
 <attribute name="VALUE" x="-4.445" y="-24.4475" size="1.27" layer="27" rot="R90"/>
 </element>
-<element name="R6" library="rcl" library_urn="urn:adsk.eagle:library:334" package="R0603" package3d_urn="urn:adsk.eagle:package:23555/3" value="1180k" x="-6.35" y="-26.9875" smashed="yes" rot="R90">
+<element name="R6" library="rcl" library_urn="urn:adsk.eagle:library:334" package="R0603" package3d_urn="urn:adsk.eagle:package:23555/3" value="18k" x="-6.35" y="-26.9875" smashed="yes" rot="R90">
 <attribute name="NAME" x="-5.08" y="-26.9875" size="0.8" layer="25" ratio="10" rot="R90" align="center"/>
 <attribute name="POPULARITY" value="77" x="-6.35" y="-26.9875" size="1.778" layer="27" rot="R90" display="off"/>
@@
 <attribute name="VALUE" x="-4.445" y="-27.6225" size="1.27" layer="27" rot="R90"/>
 </element>
-<element name="R7" library="rcl" library_urn="urn:adsk.eagle:library:334" package="R0603" package3d_urn="urn:adsk.eagle:package:23555/3" value="34k" x="-3.81" y="-28.2575" smashed="yes" rot="R90">
+<element name="R7" library="rcl" library_urn="urn:adsk.eagle:library:334" package="R0603" package3d_urn="urn:adsk.eagle:package:23555/3" value="2k" x="-3.81" y="-28.2575" smashed="yes" rot="R90">
 <attribute name="NAME" x="-2.54" y="-28.2575" size="0.8" layer="25" ratio="10" rot="R90" align="center"/>
 <attribute name="POPULARITY" value="77" x="-8.89" y="-28.2575" size="1.778" layer="27" rot="R90" display="off"/>
@@
 <attribute name="VALUE" x="-1.905" y="-28.8925" size="1.27" layer="27" rot="R90"/>
 </element>
-<element name="R8" library="rcl" library_urn="urn:adsk.eagle:library:334" package="R0603" package3d_urn="urn:adsk.eagle:package:23555/3" value="86.6k" x="-6.35" y="-30.1625" smashed="yes" rot="R90">
+<element name="R8" library="rcl" library_urn="urn:adsk.eagle:library:334" package="R0603" package3d_urn="urn:adsk.eagle:package:23555/3" value="1k" x="-6.35" y="-30.1625" smashed="yes" rot="R90">
 <attribute name="NAME" x="-5.08" y="-30.1625" size="0.8" layer="25" ratio="10" rot="R90" align="center"/>
 <attribute name="POPULARITY" value="77" x="-1.27" y="-30.1625" size="1.778" layer="27" rot="R90" display="off"/>
